File: Capacitor_Boards/capacitor_motherboard/cap_motherboad/cap_motherboad.kicad_sch (KiCad schematic)
At the start: 14 parts, among them J1 Conn_01x02_Female, J10 Conn_01x02_Female, J11 Conn_01x02_Female, J12 Conn_01x02_Female, J2 Conn_01x02_Female, J3 Conn_01x02_Female, J4 Conn_01x02_Female, J5 Conn_01x02_Female, J6 Conn_01x02_Female, J7 Conn_01x02_Female, J8 Conn_01x02_Female, J9 Conn_01x02_Female

Commit message: Finalized boards
Parts:
- removed J1, J2, J3, J4, J5, J6: Conn_01x02_Female, Connector_PinSocket_2.54mm:PinSocket_1x02_P2.54mm_Vertical, symbol Connector:Conn_01x02_Female
- removed J10, J11, J12, J7, J8, J9: Conn_01x02_Female, symbol Connector:Conn_01x02_Female
- added H1: (no value), symbol Mechanical:MountingHole
- added H2, H3, H4, H5: MountingHole, MountingHole:MountingHole_3.2mm_M3, symbol Mechanical:MountingHole
- added J1, J10, J11, J12, J2, J3, J4, J5, J6, J7, J8, J9: Conn_01x05, Connector_PinSocket_2.54mm:PinSocket_1x05_P2.54mm_Vertical, symbol Connector_Generic:Conn_01x05
Connections:
- net GND: now also J10.1 (Pin_1), J10.2 (Pin_2), J10.3 (Pin_3), J10.4 (Pin_4), J10.5 (Pin_5), J11.1 (Pin_1), J11.2 (Pin_2), J11.3 (Pin_3), J11.4 (Pin_4), J11.5 (Pin_5), J12.1 (Pin_1), J12.2 (Pin_2), J12.3 (Pin_3), J12.4 (Pin_4), J12.5 (Pin_5)
- net at QLA1.1 (In): now also J1.1 (Pin_1), J1.2 (Pin_2), J1.3 (Pin_3), J1.4 (Pin_4), J1.5 (Pin_5), J2.1 (Pin_1), J2.2 (Pin_2), J2.3 (Pin_3), J2.4 (Pin_4), J2.5 (Pin_5), J3.1 (Pin_1), J3.2 (Pin_2), J3.3 (Pin_3), J3.4 (Pin_4), J3.5 (Pin_5)
- net at SMA1.1 (In): now also J4.1 (Pin_1), J4.2 (Pin_2), J4.3 (Pin_3), J4.4 (Pin_4), J4.5 (Pin_5), J5.1 (Pin_1), J5.2 (Pin_2), J5.3 (Pin_3), J5.4 (Pin_4), J5.5 (Pin_5), J6.1 (Pin_1), J6.2 (Pin_2), J6.3 (Pin_3), J6.4 (Pin_4), J6.5 (Pin_5), J7.1 (Pin_1), J7.2 (Pin_2), J7.3 (Pin_3), J7.4 (Pin_4), J7.5 (Pin_5), J8.1 (Pin_1), J8.2 (Pin_2), J8.3 (Pin_3), J8.4 (Pin_4), J8.5 (Pin_5), J9.1 (Pin_1), J9.2 (Pin_2), J9.3 (Pin_3), J9.4 (Pin_4), J9.5 (Pin_5)
Other:
- moved on the sheet: QLA1, SMA1
